Commit message: ros2_ur5_interfaces_29/01/25

File: ros2_ws/src/ros2_ur5_interface/models/ur_gz.ros2_control.xacro (robot description, xacro)
@@ -6,5 +6,5 @@
     tf_prefix
     transmission_hw_interface:=hardware_interface/PositionJointInterface
-    initial_positions:=${dict(shoulder_pan_joint=-1.60,shoulder_lift_joint=-1.72,elbow_joint=-2.20,wrist_1_joint=-0.81,wrist_2_joint=1.60,wrist_3_joint=-0.03)}
+    initial_positions:=${dict(shoulder_pan_joint=-1.60,shoulder_lift_joint=-1.72,elbow_joint=-2.20,wrist_1_joint=-0.81,wrist_2_joint=-1.60,wrist_3_joint=-0.03)}
     ">
     <!-- Add URDF transmission elements (for ros_control) -->

File: ros2_ws/src/ros2_ur5_interface/models/ur_gz.urdf.xacro (robot description, xacro)
@@ -24,5 +24,5 @@
     <collision>
       <geometry>
-        <box size="1.0 1.0 0.0001"/>
+        <box size="1.0 1.0 0.01"/>
       </geometry>
     </collision>
